Commit message: Fix model to match product specification

File: abb_irb6640_support/urdf/irb6640_185_280.urdf (robot description, URDF)
Before this commit: robot abb_irb6640_185_280, 11 links, 10 joints
Joints:
- joint joint_1: origin xyz=0 0 0.227 rpy=0 0 0 -> xyz=0 0 0 rpy=0 0 0
- joint joint_2: origin xyz=0.322 0.03 0.551 rpy=0 0 0 -> xyz=0.320 0 0.780 rpy=0 0 0
- joint joint_3: origin xyz=0 -0.2 1.07 rpy=0 0 0 -> xyz=0 0 1.075 rpy=0 0 0
- joint joint_4: origin xyz=-0.275 0.181 0.2 rpy=0 0 0 -> xyz=0 0 0.2 rpy=0 0 0
- joint joint_5: origin xyz=1.67 0 0  rpy=0 0 0 -> xyz=1.392 0 0  rpy=0 0 0
- joint joint_6: origin xyz=0.153 0 0  rpy=0 0 0 -> xyz=0.2 0 0  rpy=0 0 0
- joint joint_6-tool0: origin xyz=.055 0 0 rpy=0 1.57079632679 0 -> xyz=0 0 0 rpy=0 1.57079632679 0
- joint joint_cylinder: limit lower=-2.96705973 upper=2.96705973 effort=0 velocity=0 -> (none); mimic (none) -> joint=joint_2 multiplier=-0.25; origin xyz=-0.365 -0.1895 0.405 rpy=0 -0.170 0 -> xyz=-0.3647 0 0.6345 rpy=0 0 0; type fixed -> continuous
- joint joint_piston: axis 1 0 0 -> 0 1 0; limit lower=0 upper=0.6 effort=0 velocity=0 -> (none); mimic (none) -> joint=joint_2 multiplier=-1.25; origin xyz=0.475 0 0 rpy=0 0 0 -> xyz=-0.22 0 -0.0672 rpy=0 0 0; parent link_cylinder -> link_2; type fixed -> continuous

File: abb_irb6640_support/urdf/irb6640_185_280_macro.xacro (robot description, xacro)
@@ -14,9 +14,6 @@
       <visual name="visual">
         <geometry>
-          <mesh filename="package://abb_irb6640_support/meshes/irb6640_185_280/visual/base_link.stl"/>
+          <mesh filename="package://abb_irb6640_support/meshes/irb6640_185_280/visual/base_link.dae"/>
         </geometry>
-        <material name="orange">
-          <color rgba="1 0.43 0 1"/>
-        </material>
       </visual>
     </link>
@@ -30,7 +27,6 @@
       <visual name="visual">
         <geometry>
-          <mesh filename="package://abb_irb6640_support/meshes/irb6640_185_280/visual/link_1.stl"/>
+          <mesh filename="package://abb_irb6640_support/meshes/irb6640_185_280/visual/link_1.dae"/>
         </geometry>
-        <material name="orange"/>
       </visual>
     </link>
@@ -44,7 +40,6 @@
       <visual name="visual">
         <geometry>
-          <mesh filename="package://abb_irb6640_support/meshes/irb6640_185_280/visual/link_2.stl"/>
+          <mesh filename="package://abb_irb6640_support/meshes/irb6640_185_280/visual/link_2.dae"/>
         </geometry>
-        <material name="orange"/>
       </visual>
     </link>
@@ -58,7 +53,6 @@
       <visual name="visual">
         <geometry>
-          <mesh filename="package://abb_irb6640_support/meshes/irb6640_185_280/visual/link_3.stl"/>
+          <mesh filename="package://abb_irb6640_support/meshes/irb6640_185_280/visual/link_3.dae"/>
         </geometry>
-        <material name="orange"/>
       </visual>
     </link>
@@ -68,11 +62,9 @@
           <mesh filename="package://abb_irb6640_support/meshes/irb6640_185_280/collision/link_4.stl"/>
         </geometry>
-        <material name="yellow"/>
       </collision>
       <visual name="visual">
         <geometry>
-          <mesh filename="package://abb_irb6640_support/meshes/irb6640_185_280/visual/link_4.stl"/>
+          <mesh filename="package://abb_irb6640_support/meshes/irb6640_185_280/visual/link_4.dae"/>
         </geometry>
-        <material name="orange"/>
       </visual>
     </link>
@@ -86,7 +78,6 @@
       <visual name="visual">
         <geometry>
-          <mesh filename="package://abb_irb6640_support/meshes/irb6640_185_280/visual/link_5.stl"/>
+          <mesh filename="package://abb_irb6640_support/meshes/irb6640_185_280/visual/link_5.dae"/>
         </geometry>
-        <material name="orange"/>
       </visual>
     </link>
@@ -100,7 +91,6 @@
       <visual name="visual">
         <geometry>
-          <mesh filename="package://abb_irb6640_support/meshes/irb6640_185_280/visual/link_6.stl"/>
+          <mesh filename="package://abb_irb6640_support/meshes/irb6640_185_280/visual/link_6.dae"/>
         </geometry>
-        <material name="orange"/>
       </visual>
     </link>
@@ -110,5 +100,5 @@
       <collision name="collision">
         <geometry>
-          <mesh filename="package://abb_irb6640_support/meshes/irb6640_185_280/collision/cylinder.stl"/>
+          <mesh filename="package://abb_irb6640_support/meshes/irb6640_185_280/collision/cylinder_link.stl"/>
         </geometry>
         <material name="yellow"/>
@@ -116,7 +106,6 @@
       <visual name="visual">
         <geometry>
-          <mesh filename="package://abb_irb6640_support/meshes/irb6640_185_280/visual/cylinder.stl"/>
+          <mesh filename="package://abb_irb6640_support/meshes/irb6640_185_280/visual/cylinder_link.dae"/>
         </geometry>
-        <material name="orange"/>
       </visual>
     </link>
@@ -124,5 +113,5 @@
       <collision name="collision">
         <geometry>
-          <mesh filename="package://abb_irb6640_support/meshes/irb6640_185_280/collision/piston.stl"/>
+          <mesh filename="package://abb_irb6640_support/meshes/irb6640_185_280/collision/piston_link.stl"/>
         </geometry>
         <material name="yellow"/>
@@ -130,7 +119,6 @@
       <visual name="visual">
         <geometry>
-          <mesh filename="package://abb_irb6640_support/meshes/irb6640_185_280/visual/piston.stl"/>
+          <mesh filename="package://abb_irb6640_support/meshes/irb6640_185_280/visual/piston_link.dae"/>
         </geometry>
-        <material name="orange"/>
       </visual>
     </link>
@@ -138,5 +126,5 @@
     <!-- joint list -->
     <joint type="revolute" name="${prefix}joint_1">
-      <origin xyz="0 0 0.227" rpy="0 0 0"/>
+      <origin xyz="0 0 0" rpy="0 0 0"/>
       <axis xyz="0 0 1"/>
       <parent link="${prefix}base_link"/>
@@ -145,5 +133,5 @@
     </joint>
     <joint type="revolute" name="${prefix}joint_2">
-      <origin xyz="0.322 0.03 0.551" rpy="0 0 0"/>
+      <origin xyz="0.320 0 0.780" rpy="0 0 0"/>
       <axis xyz="0 1 0"/>
       <parent link="${prefix}link_1"/>
@@ -152,5 +140,5 @@
     </joint>
     <joint type="revolute" name="${prefix}joint_3">
-      <origin xyz="0 -0.2 1.07" rpy="0 0 0"/>
+      <origin xyz="0 0 1.075" rpy="0 0 0"/>
       <axis xyz="0 1 0"/>
       <parent link="${prefix}link_2"/>
@@ -159,5 +147,5 @@
     </joint>
     <joint type="revolute" name="${prefix}joint_4">
-      <origin xyz="-0.275 0.181 0.2" rpy="0 0 0"/>
+      <origin xyz="0 0 0.2" rpy="0 0 0"/>
       <axis xyz="1 0 0"/>
       <parent link="${prefix}link_3"/>
@@ -166,5 +154,5 @@
     </joint>
     <joint type="revolute" name="${prefix}joint_5">
-      <origin xyz="1.67 0 0 " rpy="0 0 0"/>
+      <origin xyz="1.392 0 0 " rpy="0 0 0"/>
       <axis xyz="0 1 0"/>
       <parent link="${prefix}link_4"/>
@@ -173,5 +161,5 @@
     </joint>
     <joint type="revolute" name="${prefix}joint_6">
-      <origin xyz="0.153 0 0 " rpy="0 0 0"/>
+      <origin xyz="0.2 0 0 " rpy="0 0 0"/>
       <axis xyz="1 0 0"/>
       <parent link="${prefix}link_5"/>
@@ -182,19 +170,19 @@
       <parent link="${prefix}link_6"/>
       <child link="${prefix}tool0"/>
-      <origin xyz=".055 0 0" rpy="0 1.57079632679 0"/>
+      <origin xyz="0 0 0" rpy="0 1.57079632679 0"/>
     </joint>
-    <joint type="fixed" name="${prefix}joint_cylinder">
-      <origin xyz="-0.365 -0.1895 0.405" rpy="0 -0.170 0"/>
+    <joint type="continuous" name="${prefix}joint_cylinder">
+      <origin xyz="-0.3647 0 0.6345" rpy="0 0 0"/>
       <axis xyz="0 1 0"/>
       <parent link="${prefix}link_1"/>
       <child link="${prefix}link_cylinder"/>
-      <limit effort="0" lower="-2.96705973" upper="2.96705973" velocity="0"/>
+      <mimic joint="${prefix}joint_2" multiplier="-0.25"/>
     </joint>
-    <joint type="fixed" name="${prefix}joint_piston">
-      <origin xyz="0.475 0 0" rpy="0 0 0"/>
-      <axis xyz="1 0 0"/>
-      <parent link="${prefix}link_cylinder"/>
+    <joint type="continuous" name="${prefix}joint_piston">
+      <origin xyz="-0.22 0 -0.0672" rpy="0 0 0"/>
+      <axis xyz="0 1 0"/>
+      <parent link="${prefix}link_2"/>
       <child link="${prefix}link_piston"/>
-      <limit effort="0" lower="0" upper="0.6" velocity="0"/>
+      <mimic joint="${prefix}joint_2" multiplier="-1.25"/>
     </joint>
     <!-- end of joint list -->

Commit message: Fix errors, requested changes and update moveit config package

File: abb_irb6640_support/urdf/irb6640_185_280.urdf (robot description, URDF)
Before this commit: robot abb_irb6640_185_280, 11 links, 10 joints
Joints:
- joint joint_1: origin xyz=0 0 0 rpy=0 0 0 -> xyz=0 0 0.780 rpy=0 0 0
- joint joint_2: origin xyz=0.320 0 0.780 rpy=0 0 0 -> xyz=0.320 0 0 rpy=0 0 0
- joint joint_cylinder: origin xyz=-0.3647 0 0.6345 rpy=0 0 0 -> xyz=-0.3647 0 -0.1455 rpy=0 0 0

File: abb_irb6640_support/urdf/irb6640_185_280_macro.xacro (robot description, xacro)
@@ -8,7 +8,4 @@
           <mesh filename="package://abb_irb6640_support/meshes/irb6640_185_280/collision/base_link.stl"/>
         </geometry>
-        <material name="yellow">
-          <color rgba="0 1 1 1"/>
-        </material>
       </collision>
       <visual name="visual">
@@ -16,4 +13,7 @@
           <mesh filename="package://abb_irb6640_support/meshes/irb6640_185_280/visual/base_link.dae"/>
         </geometry>
+        <material name="yellow">
+          <color rgba="1 1 0 1"/>
+        </material>
       </visual>
     </link>
@@ -23,5 +23,4 @@
           <mesh filename="package://abb_irb6640_support/meshes/irb6640_185_280/collision/link_1.stl"/>
         </geometry>
-        <material name="yellow"/>
       </collision>
       <visual name="visual">
@@ -29,4 +28,5 @@
           <mesh filename="package://abb_irb6640_support/meshes/irb6640_185_280/visual/link_1.dae"/>
         </geometry>
+        <material name="yellow"/>
       </visual>
     </link>
@@ -36,5 +36,4 @@
           <mesh filename="package://abb_irb6640_support/meshes/irb6640_185_280/collision/link_2.stl"/>
         </geometry>
-        <material name="yellow"/>
       </collision>
       <visual name="visual">
@@ -42,4 +41,5 @@
           <mesh filename="package://abb_irb6640_support/meshes/irb6640_185_280/visual/link_2.dae"/>
         </geometry>
+        <material name="yellow"/>
       </visual>
     </link>
@@ -49,5 +49,4 @@
           <mesh filename="package://abb_irb6640_support/meshes/irb6640_185_280/collision/link_3.stl"/>
         </geometry>
-        <material name="yellow"/>
       </collision>
       <visual name="visual">
@@ -55,4 +54,5 @@
           <mesh filename="package://abb_irb6640_support/meshes/irb6640_185_280/visual/link_3.dae"/>
         </geometry>
+        <material name="yellow"/>
       </visual>
     </link>
@@ -67,4 +67,5 @@
           <mesh filename="package://abb_irb6640_support/meshes/irb6640_185_280/visual/link_4.dae"/>
         </geometry>
+        <material name="yellow"/>
       </visual>
     </link>
@@ -74,5 +75,4 @@
           <mesh filename="package://abb_irb6640_support/meshes/irb6640_185_280/collision/link_5.stl"/>
         </geometry>
-        <material name="yellow"/>
       </collision>
       <visual name="visual">
@@ -80,4 +80,5 @@
           <mesh filename="package://abb_irb6640_support/meshes/irb6640_185_280/visual/link_5.dae"/>
         </geometry>
+        <material name="yellow"/>
       </visual>
     </link>
@@ -87,5 +88,4 @@
           <mesh filename="package://abb_irb6640_support/meshes/irb6640_185_280/collision/link_6.stl"/>
         </geometry>
-        <material name="yellow"/>
       </collision>
       <visual name="visual">
@@ -93,4 +93,5 @@
           <mesh filename="package://abb_irb6640_support/meshes/irb6640_185_280/visual/link_6.dae"/>
         </geometry>
+        <material name="yellow"/>
       </visual>
     </link>
@@ -102,5 +103,4 @@
           <mesh filename="package://abb_irb6640_support/meshes/irb6640_185_280/collision/cylinder_link.stl"/>
         </geometry>
-        <material name="yellow"/>
       </collision>
       <visual name="visual">
@@ -108,4 +108,5 @@
           <mesh filename="package://abb_irb6640_support/meshes/irb6640_185_280/visual/cylinder_link.dae"/>
         </geometry>
+        <material name="yellow"/>
       </visual>
     </link>
@@ -115,5 +116,4 @@
           <mesh filename="package://abb_irb6640_support/meshes/irb6640_185_280/collision/piston_link.stl"/>
         </geometry>
-        <material name="yellow"/>
       </collision>
       <visual name="visual">
@@ -121,4 +121,5 @@
           <mesh filename="package://abb_irb6640_support/meshes/irb6640_185_280/visual/piston_link.dae"/>
         </geometry>
+        <material name="yellow"/>
       </visual>
     </link>
@@ -126,5 +127,5 @@
     <!-- joint list -->
     <joint type="revolute" name="${prefix}joint_1">
-      <origin xyz="0 0 0" rpy="0 0 0"/>
+      <origin xyz="0 0 0.780" rpy="0 0 0"/>
       <axis xyz="0 0 1"/>
       <parent link="${prefix}base_link"/>
@@ -133,5 +134,5 @@
     </joint>
     <joint type="revolute" name="${prefix}joint_2">
-      <origin xyz="0.320 0 0.780" rpy="0 0 0"/>
+      <origin xyz="0.320 0 0" rpy="0 0 0"/>
       <axis xyz="0 1 0"/>
       <parent link="${prefix}link_1"/>
@@ -173,5 +174,5 @@
     </joint>
     <joint type="continuous" name="${prefix}joint_cylinder">
-      <origin xyz="-0.3647 0 0.6345" rpy="0 0 0"/>
+      <origin xyz="-0.3647 0 -0.1455" rpy="0 0 0"/>
       <axis xyz="0 1 0"/>
       <parent link="${prefix}link_1"/>
