Commit message: Update visual meshes to collada file

File: abb_irb2400_support/urdf/irb2400_macro.xacro (robot description, xacro)
@@ -7,9 +7,6 @@
             <origin xyz="0 0 0" rpy="0 0 0"/>
             <geometry>
-                <mesh filename="package://abb_irb2400_support/meshes/irb2400/visual/base_link.stl"/>
+                <mesh filename="package://abb_irb2400_support/meshes/irb2400/visual/base_link.dae"/>
             </geometry>
-            <material name="abb_orange">
-                <color rgba="1 0.43 0 1"/>
-            </material>
         </visual>
         <collision>
@@ -26,7 +23,6 @@
             <origin xyz="0 0 0" rpy="0 0 0"/>
             <geometry>
-                <mesh filename="package://abb_irb2400_support/meshes/irb2400/visual/link_1.stl"/>
+                <mesh filename="package://abb_irb2400_support/meshes/irb2400/visual/link_1.dae"/>
             </geometry>
-            <material name="abb_orange"/>
         </visual>
         <collision>
@@ -42,7 +38,6 @@
             <origin xyz="0 0 0" rpy="0 0 0"/>
             <geometry>
-                <mesh filename="package://abb_irb2400_support/meshes/irb2400/visual/link_2.stl"/>
+                <mesh filename="package://abb_irb2400_support/meshes/irb2400/visual/link_2.dae"/>
             </geometry>
-            <material name="abb_orange"/>
         </visual>
         <collision>
@@ -58,7 +53,6 @@
             <origin xyz="0 0 0" rpy="0 0 0"/>
             <geometry>
-                <mesh filename="package://abb_irb2400_support/meshes/irb2400/visual/link_3.stl"/>
+                <mesh filename="package://abb_irb2400_support/meshes/irb2400/visual/link_3.dae"/>
             </geometry>
-            <material name="abb_orange"/>
         </visual>
         <collision>
@@ -74,7 +68,6 @@
             <origin xyz="0 0 0" rpy="0 0 0"/>
             <geometry>
-                <mesh filename="package://abb_irb2400_support/meshes/irb2400/visual/link_4.stl"/>
+                <mesh filename="package://abb_irb2400_support/meshes/irb2400/visual/link_4.dae"/>
             </geometry>
-            <material name="abb_orange"/>
         </visual>
         <collision>
@@ -90,7 +83,6 @@
             <origin xyz="0 0 0" rpy="0 0 0"/>
             <geometry>
-                <mesh filename="package://abb_irb2400_support/meshes/irb2400/visual/link_5.stl"/>
+                <mesh filename="package://abb_irb2400_support/meshes/irb2400/visual/link_5.dae"/>
             </geometry>
-            <material name="abb_orange"/>
         </visual>
         <collision>
@@ -106,7 +98,6 @@
             <origin xyz="0 0 0" rpy="0 0 0"/>
             <geometry>
-                <mesh filename="package://abb_irb2400_support/meshes/irb2400/visual/link_6.stl"/>
+                <mesh filename="package://abb_irb2400_support/meshes/irb2400/visual/link_6.dae"/>
             </geometry>
-            <material name="abb_orange"/>
         </visual>
         <collision>

File: abb_irb5400_support/urdf/irb5400_macro.xacro (robot description, xacro)
@@ -6,9 +6,6 @@
         <visual>
             <geometry>
-                <mesh filename="package://abb_irb5400_support/meshes/irb5400/visual/base_link.stl"/>
+                <mesh filename="package://abb_irb5400_support/meshes/irb5400/visual/base_link.dae"/>
             </geometry>
-            <material name="orange">
-                <color rgba="1 0.43 0 1"/>
-            </material>
         </visual>
         <collision>
@@ -24,7 +21,6 @@
         <visual>
             <geometry>
-                <mesh filename="package://abb_irb5400_support/meshes/irb5400/visual/link_1.stl"/>
+                <mesh filename="package://abb_irb5400_support/meshes/irb5400/visual/link_1.dae"/>
             </geometry>
-            <material name="orange"/>
         </visual>
         <collision>
@@ -38,9 +34,6 @@
         <visual>
             <geometry>
-                <mesh filename="package://abb_irb5400_support/meshes/irb5400/visual/link_2.stl"/>
+                <mesh filename="package://abb_irb5400_support/meshes/irb5400/visual/link_2.dae"/>
             </geometry>
-            <material name="lt_black">
-                <color rgba="0.3 0.3 0.3 1"/>
-            </material>
         </visual>
         <collision>
@@ -54,7 +47,6 @@
         <visual>
             <geometry>
-                <mesh filename="package://abb_irb5400_support/meshes/irb5400/visual/link_3.stl"/>
+                <mesh filename="package://abb_irb5400_support/meshes/irb5400/visual/link_3.dae"/>
             </geometry>
-            <material name="orange"/>
         </visual>
         <collision>
@@ -68,7 +60,6 @@
         <visual>
             <geometry>
-                <mesh filename="package://abb_irb5400_support/meshes/irb5400/visual/link_4.stl"/>
+                <mesh filename="package://abb_irb5400_support/meshes/irb5400/visual/link_4.dae"/>
             </geometry>
-            <material name="lt_black"/>
         </visual>
         <collision>
@@ -82,7 +73,6 @@
         <visual>
             <geometry>
-                <mesh filename="package://abb_irb5400_support/meshes/irb5400/visual/link_5.stl"/>
+                <mesh filename="package://abb_irb5400_support/meshes/irb5400/visual/link_5.dae"/>
             </geometry>
-            <material name="lt_black"/>
         </visual>
         <collision>
@@ -96,7 +86,6 @@
         <visual>
             <geometry>
-                <mesh filename="package://abb_irb5400_support/meshes/irb5400/visual/link_5b.stl"/>
+                <mesh filename="package://abb_irb5400_support/meshes/irb5400/visual/link_5b.dae"/>
             </geometry>
-            <material name="lt_black"/>
         </visual>
         <collision>
@@ -110,7 +99,6 @@
         <visual>
             <geometry>
-                <mesh filename="package://abb_irb5400_support/meshes/irb5400/visual/link_6.stl"/>
+                <mesh filename="package://abb_irb5400_support/meshes/irb5400/visual/link_6.dae"/>
             </geometry>
-            <material name="lt_black"/>
         </visual>
         <collision>
